File: can-sensor-board.kicad_pcb (KiCad board)
At the start: 2 copper layers, 35 parts, among them J1 I2C_STANDARDQWIIC, J2 I2C_STANDARDQWIIC, J3 105314-1104, J4 105314-1104, J5 TC2030-IDC-NL, J6 Conn_01x06_Male, J7 Conn_01x07_Male, U1 STM32F072CBUx, U2 SN65HVD230DR, U3 AP7381-33Y-13, Y1 TAXM8M4RDBCCT2T

Commit message: final v1 board
Parts:
- removed C11: C_0805_25V_X5R_10u, Capacitor_SMD:C_0805_2012Metric
- removed J6: Conn_01x06_Male, Connector_PinHeader_2.54mm:PinHeader_1x06_P2.54mm_Vertical
- removed J7: Conn_01x07_Male, Connector_PinHeader_2.54mm:PinHeader_1x07_P2.54mm_Vertical
- added H1: Mounting Hole, MountingHole:MountingHole_3.2mm_M3, F.Cu at (235.0, 111.0)
- added H2: Mounting Hole, MountingHole:MountingHole_3.2mm_M3, F.Cu at (211.0, 76.0)
- added H3: Mounting Hole, MountingHole:MountingHole_3.2mm_M3, F.Cu at (235.0, 76.0)
- added H4: Mounting Hole, MountingHole:MountingHole_3.2mm_M3, F.Cu at (211.0, 111.0)
- added P1: TC2030-IDC-NL, Connector:Tag-Connect_TC2030-IDC-NL_2x03_P1.27mm_Vertical, F.Cu at (212.2, 99.5)
- added TP_3V1: TestPoint_Small, footprints:TestPoint_Pad_D1.00mm, F.Cu at (234.5, 90.0)
- added TP_GND1: TestPoint_Small, footprints:TestPoint_Pad_D1.00mm, F.Cu at (236.5, 90.0)
- D4: value LED_0603_Red -> LED_0603_Green
- J1, J2: value I2C_STANDARDQWIIC -> 105314-1104; footprint Connectors:1X04_1MM_RA -> footprints:Molex_Nano-Fit_105314-xx04_2x02_P2.50mm_Horizontal
- J3, J4: value 105314-1104 -> I2C_QWIIC; footprint Connector_Molex:Molex_Nano-Fit_105314-xx04_2x02_P2.50mm_Horizontal -> footprints:JST_SH_SM04B-SRSS-TB_1x04-1MP_P1.00mm_Horizontal
- J5: value TC2030-IDC-NL -> Conn_02x05_Odd_Even; footprint Connector:Tag-Connect_TC2030-IDC-NL_2x03_P1.27mm_Vertical -> Connector_PinHeader_2.54mm:PinHeader_2x05_P2.54mm_Vertical
- R7: value R_0402_330R_1 -> R_0402_1k_1
- R8: value R_0402_330R_1 -> R_0402_2k_1
- moved D2 154.6 mm to (234.5, 86.5), turned to 90 degrees
- moved C9 152.7 mm to (228.4, 93.9)
- moved C10 143.6 mm to (217.7, 98.6), turned to 90 degrees
- moved C3 141.7 mm to (229.5, 88.8), turned to 90 degrees
- moved R7 137.8 mm to (231.2, 94.5), turned to 180 degrees
- moved U3 137.5 mm to (225.8, 88.0), turned to 90 degrees
- moved J2 131.4 mm to (226.0, 83.8), turned to 90 degrees
- moved Y1 130.4 mm to (230.4, 98.4)
- moved C7 129.4 mm to (219.7, 90.8)
- moved D3 128.5 mm to (232.0, 88.5), turned to 90 degrees
- moved C8 128.1 mm to (226.2, 100.6), turned to 180 degrees
- moved C5 128.0 mm to (227.7, 98.5), turned to 270 degrees
- moved U1 127.8 mm to (222.7, 95.7), turned to 180 degrees
- moved J5 127.3 mm to (217.9, 106.0), turned to 90 degrees
- moved D4 125.0 mm to (234.2, 94.5), turned to 180 degrees
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Connections:
- net Net-(C3-Pad1) renamed /VIN_PROT
- J1 pad 1: GND -> /CANH
- J1 pad 2: 3V3 -> /CANL
- J1 pad 3: I2C_1_SDA -> /VIN
- J1 pad 4: I2C_1_SCL -> GND
- J2 pad 1: GND -> /CANH
- J2 pad 2: 3V3 -> /CANL
- J2 pad 3: I2C_2_SDA -> /VIN
- J2 pad 4: I2C_2_SCL -> GND
- J3 pad 1: /VIN -> GND
- J3 pad 2: /CANL -> 3V3
- J3 pad 3: GND -> I2C_1_SDA
- J3 pad 4: /CANH -> I2C_1_SCL
- J4 pad 1: /VIN -> GND
- J4 pad 2: /CANL -> 3V3
- J4 pad 3: GND -> I2C_2_SDA
- J4 pad 4: /CANH -> I2C_2_SCL
- J5 pad 2: SWDIO -> Net-(J5-Pad2)
- J5 pad 3: nRESET -> GND
- J5 pad 4: SWCLK -> Net-(J5-Pad4)
- J5 pad 6: (no net) -> Net-(J5-Pad6)
- R7 pad 2: /LED_1 -> 3V3
- R8 pad 2: /LED_2 -> /STATUS_LED
- U1 pad 10: /LED_1 -> (no net)
- U1 pad 11: /LED_2 -> (no net)
- U1 pad 12: Net-(J6-Pad1) -> /STATUS_LED
- U1 pad 13: Net-(J6-Pad2) -> (no net)
- U1 pad 14: Net-(J6-Pad3) -> (no net)
- U1 pad 15: Net-(J6-Pad4) -> (no net)
- U1 pad 16: Net-(J6-Pad5) -> (no net)
- U1 pad 17: Net-(J6-Pad6) -> (no net)
- U1 pad 39: (no net) -> Net-(J5-Pad2)
- U1 pad 40: (no net) -> Net-(J5-Pad4)
- U1 pad 41: (no net) -> Net-(J5-Pad6)
- U1 pad 42: I2C_1_SCL -> Net-(J5-Pad8)
- U1 pad 43: I2C_1_SDA -> Net-(J5-Pad10)
- U1 pad 45: (no net) -> I2C_1_SCL
- U1 pad 46: (no net) -> I2C_1_SDA
Routing:
- net 3V3: track 0.00 -> 121.3 mm, vias 0 -> 4
- net GND: track 0.00 -> 51.4 mm, vias 0 -> 28
- net I2C_2_SDA: track 0.00 -> 27.2 mm, vias 0 -> 2
- net I2C_2_SCL: track 0.00 -> 26.6 mm, vias 0 -> 2
- net /VIN: track 0.00 -> 25.0 mm
- net nRESET: track 0.00 -> 21.9 mm, vias 0 -> 2
- net I2C_1_SDA: track 0.00 -> 20.8 mm
- net I2C_1_SCL: track 0.00 -> 17.0 mm
- net /CANH: track 5.73 -> 18.5 mm
- net /CANL: track 5.52 -> 18.1 mm
- net CAN_EN: track 0.00 -> 12.3 mm, vias 0 -> 2
- net SWCLK: track 0.00 -> 11.7 mm
- net CAN_TX: track 0.00 -> 10.1 mm
- net Net-(J5-Pad10): track 0.00 -> 10.0 mm
- net SWDIO: track 0.00 -> 9.58 mm
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- added copper zone on F.Cu, net 3V3
- added copper zone on B.Cu, net GND
- added copper zone on F.Cu, net GND
Other:
- board outline added: 32 x 44 mm
- board text added: "1"
- board text added: "By Cammiboi V1"
- board text added: "CAN 2 QWIIC"
- board text added: "CH"
- board text added: "CL"
- board text added: "GND"
- board text added: "VIN"
- board text removed: "ENCLOSURE OUTLINE"
