File: can-sensor-board.sch (KiCad schematic (older format))
At the start: 37 parts, among them J1 105314-1104, J2 105314-1104, J3 I2C_STANDARDQWIIC, J4 I2C_STANDARDQWIIC, J5 Conn_01x07_Male, J6 Conn_01x06_Male, P1 TC2030-IDC-NL, U1 STM32F072CBUx, U2 SN65HVD230DR, U3 AP7381-33Y-13, Y1 TAXM8M4RDBCCT2T

Commit message: final v1 board
Parts:
- removed C11: C_0805_25V_X5R_10u, Capacitor_SMD:C_0805_2012Metric, symbol cb_Capacitors-Ceramic:C_0805_25V_X5R_10u
- removed J3, J4: I2C_STANDARDQWIIC, 1X04_1MM_RA, symbol SparkFun-Connectors:I2C_STANDARDQWIIC
- removed J5: Conn_01x07_Male, Connector_PinHeader_2.54mm:PinHeader_1x07_P2.54mm_Vertical, symbol Connector:Conn_01x07_Male
- removed J6: Conn_01x06_Male, Connector_PinHeader_2.54mm:PinHeader_1x06_P2.54mm_Vertical, symbol Connector:Conn_01x06_Male
- added H1, H2, H3, H4: Mounting Hole, MountingHole:MountingHole_3.2mm_M3, symbol Mechanical:MountingHole
- added J3, J4: I2C_QWIIC, footprints:JST_SH_SM04B-SRSS-TB_1x04-1MP_P1.00mm_Horizontal, symbol cb_Connector:I2C_QWIIC
- added J5: Conn_02x05_Odd_Even, Connector_PinHeader_2.54mm:PinHeader_2x05_P2.54mm_Vertical, symbol Connector_Generic:Conn_02x05_Odd_Even
- J1, J2: footprint Connector_Molex:Molex_Nano-Fit_105314-xx04_2x02_P2.50mm_Horizontal -> footprints:Molex_Nano-Fit_105314-xx04_2x02_P2.50mm_Horizontal
Connections:
- net 3V3: now also J3.2 (VCC), J4.2 (VCC), J5.1 (Pin_1)
- net CANH: now also J1.1, J2.1; no longer J1.4 (3), J2.4 (3)
- net GND: now also J1.4 (3), J2.4 (3), J3.1 (GND), J4.1 (GND), J5.3 (Pin_3), J5.5 (Pin_5), J5.7 (Pin_7), J5.9 (Pin_9); no longer J1.3, J2.3
- net I2C_1_SCL: now also J3.4 (SCL)
- net I2C_1_SDA: now also J3.3 (SDA)
- net I2C_2_SCL: now also J4.4 (SCL)
- net I2C_2_SDA: now also J4.3 (SDA)
- net STATUS_LED: now also U1.12 (PA2); no longer U1.10 (PA0)
- net VIN: now also J1.3, J2.3; no longer J1.1, J2.1
- net at U1.39 (PB3): now also J5.2 (Pin_2)
- net at U1.40 (PB4): now also J5.4 (Pin_4)
- net at U1.41 (PB5): now also J5.6 (Pin_6)
- net at U1.42 (PB6): now also J5.8 (Pin_8)
- net at U1.43 (PB7): now also J5.10 (Pin_10)
- no-connect marks 21 -> 22
Other:
- note removed: "1x 4u7 cap for VDD"
- moved on the sheet: D1, D5, J1, J2, R8

Commit message: final v1 submitted for review
Parts:
- H1, H2, H3, H4, J1, J2, J5, P1, TP_3V1, TP_GND1: JLCPCB_IGNORE (none) -> Yes
Changed lines of the file:
@@
 F 3 "" V 1475 1400 50  0001 C CNN
 F 4 "Molex" H 1500 2175 50  0001 C CNN "Manufacturer"
+F 5 "Yes" H 1000 1450 50  0001 C CNN "JLCPCB_IGNORE"
 	1    1000 1450
 	1    0    0    -1
@@
 F 3 "" V 1475 2000 50  0001 C CNN
 F 4 "Molex" H 1500 2775 50  0001 C CNN "Manufacturer"
+F 5 "Yes" H 1000 2050 50  0001 C CNN "JLCPCB_IGNORE"
 	1    1000 2050
 	1    0    0    -1
@@
 F 2 "Connector:Tag-Connect_TC2030-IDC-NL_2x03_P1.27mm_Vertical" H 4900 5550 50  0001 C CNN
 F 3 "https://www.tag-connect.com/wp-content/uploads/bsk-pdf-manager/2019/12/TC2030-IDC-NL-Datasheet-Rev-B.pdf" H 4900 5550 50  0001 C CNN
+F 4 "Yes" H 4900 5550 50  0001 C CNN "JLCPCB_IGNORE"
 	1    4900 5550
 	1    0    0    -1
@@
 F 2 "footprints:TestPoint_Pad_D1.00mm" H 6000 1550 50  0001 C CNN
 F 3 "~" H 6000 1550 50  0001 C CNN
+F 4 "Yes" H 5800 1550 50  0001 C CNN "JLCPCB_IGNORE"
 	1    5800 1550
 	0    1    1    0
@@
 F 2 "footprints:TestPoint_Pad_D1.00mm" H 6000 1650 50  0001 C CNN
 F 3 "~" H 6000 1650 50  0001 C CNN
+F 4 "Yes" H 5800 1650 50  0001 C CNN "JLCPCB_IGNORE"
 	1    5800 1650
 	0    1    1    0
@@
 F 2 "MountingHole:MountingHole_3.2mm_M3" H 3250 6650 50  0001 C CNN
 F 3 "~" H 3250 6650 50  0001 C CNN
+F 4 "Yes" H 3250 6650 50  0001 C CNN "JLCPCB_IGNORE"
 	1    3250 6650
 	1    0    0    -1
@@
 F 2 "MountingHole:MountingHole_3.2mm_M3" H 3250 6900 50  0001 C CNN
 F 3 "~" H 3250 6900 50  0001 C CNN
+F 4 "Yes" H 3250 6900 50  0001 C CNN "JLCPCB_IGNORE"
 	1    3250 6900
 	1    0    0    -1
@@
 F 2 "MountingHole:MountingHole_3.2mm_M3" H 4200 6650 50  0001 C CNN
 F 3 "~" H 4200 6650 50  0001 C CNN
+F 4 "Yes" H 4200 6650 50  0001 C CNN "JLCPCB_IGNORE"
 	1    4200 6650
 	1    0    0    -1
@@
 F 2 "MountingHole:MountingHole_3.2mm_M3" H 4200 6900 50  0001 C CNN
 F 3 "~" H 4200 6900 50  0001 C CNN
+F 4 "Yes" H 4200 6900 50  0001 C CNN "JLCPCB_IGNORE"
 	1    4200 6900
 	1    0    0    -1
@@
 F 2 "Connector_PinHeader_2.54mm:PinHeader_2x05_P2.54mm_Vertical" H 5800 3950 50  0001 C CNN
 F 3 "~" H 5800 3950 50  0001 C CNN
+F 4 "Yes" H 5800 3950 50  0001 C CNN "JLCPCB_IGNORE"
 	1    5800 3950
 	1    0    0    -1
